File: PI-Shield.brd (EAGLE design)
At the start: 69.8 x 73 mm, 77 parts, among them IC1 PCF8574T, J10 T2I, J11 T2I, J12 T2I, J13 DF13-4P-1.25DSA, J14 DF13-4P-1.25DSA, J15 DF13-4P-1.25DSA, Q1 220mA/50V/3.5Ω, Q2 220mA/50V/3.5Ω, Q3 220mA/50V/3.5Ω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

Commit message: v2 Changes
Would like to formally apologize for the routing of the GPIO on the bottom of the board. It was necessary, unfortunately.
Changes: [Removed expander, added LED and Header Labels, really shitty routing.]
Parts:
- removed IC1: PCF8574T, micro-philips:SO16W
- moved J2 6.36 mm to (19.9, 35.9)
- moved J9 6.36 mm to (30.1, 32.5)
- moved R17 4.89 mm to (27.2, 22.1)
- moved D4 4.85 mm to (29.4, 22.3)
- moved C14 4.83 mm to (18.0, 12.7)
- moved R18 4.83 mm to (17.4, 7.11)
- moved R21 4.83 mm to (17.4, 9.14)
- moved R22 4.83 mm to (33.7, 12.3)
- moved R23 4.83 mm to (24.9, 11.9)
- moved R24 4.83 mm to (27.2, 13.6)
- moved U$7 4.83 mm to (26.7, 12.4)
- moved C10 4.83 mm to (18.0, 16.5)
- moved Q5 4.83 mm to (27.0, 19.3)
- moved R16 4.83 mm to (24.1, 19.3)
- moved J8 4.33 mm to (6.99, 39.5)
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Connections:
- net 3V3: no longer IC1.16
- net GND: no longer IC1.1, IC1.2, IC1.3, IC1.8
- net GPIO1: now also U$8.12; no longer IC1.4
- net GPIO2: now also U$8.16; no longer IC1.5
- net GPIO3: now also U$8.18; no longer IC1.6
- net GPIO4: now also U$8.22; no longer IC1.7
- net GPIO5: now also U$8.32; no longer IC1.9
- net GPIO6: now also U$8.40; no longer IC1.10
- net SCL: no longer IC1.14
- net SDA: no longer IC1.15
Routing:
- net GPIO6: track 12.6 -> 152.7 mm
- net GPIO5: track 6.70 -> 138.1 mm, vias 1 -> 0
- net GPIO4: track 6.19 -> 128.2 mm, vias 1 -> 0
- net GPIO3: track 6.19 -> 118.5 mm, vias 1 -> 0
- net GPIO2: track 6.14 -> 114.0 mm, vias 1 -> 0
- net GPIO1: track 6.09 -> 106.3 mm, vias 1 -> 0
- net SOL6_1: track 47.8 -> 26.7 mm, vias 0 -> 1
- net 3V3: track 221.7 -> 200.9 mm
- net SOL5_1: track 42.0 -> 24.1 mm, vias 0 -> 1
- net SOL4_1: track 37.3 -> 20.9 mm, vias 0 -> 1
- net SCL: track 142.7 -> 128.7 mm
- net SOL3_1: track 31.8 -> 18.2 mm, vias 0 -> 1
- net SOL2_1: track 26.9 -> 14.4 mm
- net PI_POWER: track 25.8 -> 15.9 mm
- net SOL1_1: track 21.5 -> 13.0 mm
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Other:
- board text added: "3.3V - GND"
- board text added: "3.3V LED"
- board text added: "5V LED"
- board text added: "BNO055"
- board text added: "CS - MISO - MOSI - CLK - GND"
- board text added: "FXOS8700 FXAS21002"
- board text added: "GND - AIN2 - 3V3 - 5V"
- board text added: "GND - SCL - SDA - 3.3V"
- board text added: "PWM - 5V - GND"

Commit message: Adjusted some labels, fixed minor errors
Parts:
- removed U$3: 6X_CONN, PI-SHIELD, Solenoid-Backplane:IPL6X2
- added U$9: 7X_CONN, PI-SHIELD, Solenoid-Backplane:IPL7X2
- moved J2 6.36 mm to (20.2, 29.6)
- moved J9 6.36 mm to (30.3, 26.2)
- moved R17 4.89 mm to (26.4, 17.3)
- moved D4 4.85 mm to (28.9, 17.4)
- moved C14 4.83 mm to (18.0, 7.90)
- moved R18 4.83 mm to (17.4, 2.29)
- moved R21 4.83 mm to (17.4, 4.32)
- moved R22 4.83 mm to (33.7, 7.52)
- moved R23 4.83 mm to (24.9, 7.11)
- moved R24 4.83 mm to (27.2, 8.76)
- moved U$7 4.83 mm to (26.7, 7.62)
- moved C10 4.83 mm to (18.0, 11.6)
- moved Q5 4.83 mm to (27.0, 14.5)
- moved R16 4.83 mm to (24.1, 14.5)
- moved J8 4.33 mm to (4.19, 36.2)
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Connections:
- net 12V: now also U$9.2, U$9.4; no longer U$3.2, U$3.4
- net 3V3: now also U$9.12; no longer U$3.12
- net 5V: now also U$9.8; no longer U$3.8
- net CAN_H: now also U$9.13
- net CAN_L: now also U$9.14
- net GND: now also U$9.10, U$9.6; no longer U$3.10, U$3.6
- net SOL1_1: now also U$9.1; no longer U$3.1
- net SOL2_1: now also U$9.3; no longer U$3.3
- net SOL3_1: now also U$9.5; no longer U$3.5
- net SOL4_1: now also U$9.7; no longer U$3.7
- net SOL5_1: now also U$9.9; no longer U$3.9
- net SOL6_1: now also U$9.11; no longer U$3.11
Routing:
- net CAN_L: track 43.0 -> 131.4 mm, vias 1 -> 2
- net CAN_H: track 43.0 -> 130.9 mm, vias 1 -> 2
- net GPIO1: track 106.3 -> 86.6 mm, vias 0 -> 3
- net GPIO2: track 114.0 -> 95.1 mm, vias 0 -> 4
- net GPIO4: track 128.2 -> 110.4 mm, vias 0 -> 2
- net GPIO3: track 118.5 -> 101.7 mm, vias 0 -> 4
- net GPIO6: track 152.7 -> 138.2 mm
- net PI_POWER: track 15.9 -> 30.0 mm
- net 5V: track 172.5 -> 185.8 mm
- net GPIO5: track 138.1 -> 126.0 mm, vias 0 -> 2
- net 3V3: track 200.9 -> 211.9 mm, vias 4 -> 5
- net 5V_RAW: track 0.00 -> 6.33 mm
- net A_INT: track 61.3 -> 66.6 mm
- net IMU_INT: track 54.7 -> 59.2 mm, vias 4 -> 1
- net AIN2: track 18.4 -> 13.8 mm
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- removed copper zone on layer 1, net 5V
- removed copper zone on layer 1, net 5V_RAW
- removed copper zone on layer 1, net PI_POWER
Other:
- board text added: "3.3V"
- board text added: "5V"
- board text added: "AIN2"
- board text added: "CAN_H"
- board text added: "CAN_L"
- board text added: "CLK"
- board text added: "CS"
- board text added: "GND"
- board text added: "MISO"
- board text added: "MOSI"
- board text added: "PWM"
- board text added: "RX"
- board text added: "SCL"
- board text added: "SDA"
- board text added: "TX"
- board text added: "X14 Pi-Shield v1 Rachel Livesay Erin Park Katherine Sandys Read Hedl 3/14/2022"
- board text removed: "3.3V - GND"
- board text removed: "3.3V LED"
- board text removed: "5V LED"
- board text removed: "BNO055"
- board text removed: "CS - MISO - MOSI - CLK - GND"
- board text removed: "FXOS8700 FXAS21002"
- board text removed: "GND - AIN2 - 3V3 - 5V"
- board text removed: "GND - SCL - SDA - 3.3V"
- board text removed: "PWM - 5V - GND"
